Commit message: Added yaml configs

File: urdf_l2/urdf/manip.urdf.xacro (robot description, xacro)
@@ -1,12 +1,17 @@
 <?xml version="1.0" encoding="utf-8"?>
 <robot xmlns:xacro="http://www.ros.org/wiki/xacro" name="manip">
-<xacro:arg name="l1" default="0.4"/>
-<xacro:arg name="r1" default="0.1"/>
-<xacro:arg name="l2" default="0.2"/>
-<xacro:arg name="r2" default="0.1"/>
-<xacro:arg name="l3" default="0.2"/>
-<xacro:arg name="r3" default="0.1"/>
-<xacro:arg name="l4" default="0.15"/>
-<xacro:arg name="aa4" default="0.1"/>
+<!-- Rozmiary czlonow -->
+<xacro:property name="sizes" value="${load_yaml('sizes.yaml')}"/>
+<!-- Stawy -->
+<xacro:property name="joints" value="${load_yaml('joints.yaml')}"/>
+<xacro:property name="j1" value="prismatic"/>
+<xacro:property name="j2" value="revolute"/>
+<xacro:property name="j3" value="revolute"/>
+<xacro:if value="${joints['fixed_joints']==True}">
+  <xacro:property name="j1" value="fixed"/>
+  <xacro:property name="j2" value="fixed"/>
+  <xacro:property name="j3" value="fixed"/>
+</xacro:if>
+<!-- Parametry DH -->
 <xacro:arg name="a1" default="0.5"/>
 <xacro:arg name="a2" default="0.5"/>
@@ -46,22 +51,22 @@
 <link name="el1">
   <visual>
-    <origin xyz="0 0 ${$(arg l1)/2}" />
+    <origin xyz="0 0 ${sizes['sizes']['l1']/2}" />
     <geometry>
-      <cylinder radius="$(arg r1)" length="$(arg l1)"/>
+      <cylinder radius="${sizes['sizes']['r1']}" length="${sizes['sizes']['l1']}"/>
     </geometry>
     <material name="white"/>
   </visual>
   <collision>
-    <origin xyz="0 0 ${$(arg l1)/2}" />
+    <origin xyz="0 0 ${sizes['sizes']['r1']/2}" />
     <geometry>
-      <cylinder radius="$(arg r1)" length="$(arg l1)"/>
+      <cylinder radius="${sizes['sizes']['r1']}" length="${sizes['sizes']['l1']}"/>
     </geometry>
     <contact_coefficients mu="0" kp="1000.0" kd="1.0"/>
   </collision>
 </link>
-<joint name="el1-el2" type="prismatic">
+<joint name="el1-el2" type="${j1}">
   <parent link="el1"/>
   <child link="el2"/>
-  <origin xyz="0 0 ${$(arg l1)+0.1}" rpy="0 0 0" />
+  <origin xyz="0 0 ${sizes['sizes']['l1']+0.1}" rpy="0 0 0" />
   <axis xyz="0 0 1" />
   <limit upper="0" lower="0.0" effort="10" velocity="10" />
@@ -74,7 +79,7 @@
   </inertial>
   <visual>
-    <origin xyz="0 0 ${$(arg l2)/2}" rpy="0 0 0" />
+    <origin xyz="0 0 ${sizes['sizes']['l2']/2}" rpy="0 0 0" />
     <geometry>
-      <cylinder radius="$(arg r2)" length="$(arg l2)"/>
+      <cylinder radius="${sizes['sizes']['r2']}" length="${sizes['sizes']['l2']}"/>
     </geometry>
     <material name="white">
@@ -83,15 +88,15 @@
   </visual>
   <collision>
-    <origin xyz="0 0 ${$(arg l2)/2}" />
+    <origin xyz="0 0 ${sizes['sizes']['l2']/2}" />
     <geometry>
-      <cylinder radius="$(arg r2)" length="$(arg l2)"/>
+      <cylinder radius="${sizes['sizes']['r2']}" length="${sizes['sizes']['l2']}"/>
     </geometry>
     <contact_coefficients mu="0" kp="1000.0" kd="1.0"/>
   </collision>
 </link>
-<joint name="el2-el3" type="revolute">
+<joint name="el2-el3" type="${j2}">
   <parent link="el2"/>
   <child link="el3"/>
-  <origin xyz="0 0 ${$(arg l2)/2}" rpy="0 0 0" />
+  <origin xyz="0 0 ${sizes['sizes']['l2']/2}" rpy="0 0 0" />
   <axis xyz="0 0 1" />
   <limit upper="0" lower="0.0" effort="10" velocity="10" />
@@ -104,7 +109,7 @@
   </inertial>
   <visual>
-    <origin xyz="${$(arg r2)+$(arg r3)} 0 0"/>
+    <origin xyz="${sizes['sizes']['r2']+sizes['sizes']['r3']} 0 0"/>
     <geometry>
-      <cylinder radius="$(arg r3)" length="$(arg l3)"/>
+      <cylinder radius="${sizes['sizes']['r3']}" length="${sizes['sizes']['l3']}"/>
     </geometry>
     <material name="white">
@@ -113,15 +118,15 @@
   </visual>
   <collision>
-    <origin xyz="${$(arg r2)+$(arg r3)} 0 0"/>
+    <origin xyz="${sizes['sizes']['r2']+sizes['sizes']['r3']} 0 0"/>
     <geometry>
-      <cylinder radius="$(arg r3)" length="$(arg l3)"/>
+      <cylinder radius="${sizes['sizes']['r3']}" length="${sizes['sizes']['l3']}"/>
     </geometry>
     <contact_coefficients mu="0" kp="1000.0" kd="1.0"/>
   </collision>
 </link>
-<joint name="el3-tool" type="revolute">
+<joint name="el3-tool" type="${j3}">
   <parent link="el3"/>
   <child link="tool"/>
-  <origin xyz="${2*$(arg r3)} 0 0" rpy="0 0 0" />
+  <origin xyz="${2*sizes['sizes']['r3']} 0 0" rpy="0 0 0" />
   <axis xyz="0 0 1" />
   <limit upper="0" lower="0.0" effort="10" velocity="10" />
@@ -134,7 +139,7 @@
   </inertial>
   <visual>
-    <origin xyz="${$(arg l4)/2+$(arg r3)} 0 0" />
+    <origin xyz="${sizes['sizes']['l4']/2+sizes['sizes']['r3']} 0 0" />
     <geometry>
-      <box size="$(arg l4) $(arg aa4) $(arg aa4)"/>
+      <box size="${sizes['sizes']['l4']} ${sizes['sizes']['aa4']} ${sizes['sizes']['aa4']}"/>
     </geometry>
     <material name="white">
@@ -143,7 +148,7 @@
   </visual>
   <collision>
-    <origin xyz="${$(arg l4)/2+$(arg r3)} 0 0" />
+    <origin xyz="${sizes['sizes']['l4']/2+sizes['sizes']['r3']} 0 0" />
     <geometry>
-      <box size="$(arg l4) $(arg aa4) $(arg aa4)"/>
+      <box size="${sizes['sizes']['l4']} ${sizes['sizes']['aa4']} ${sizes['sizes']['aa4']}"/>
     </geometry>
     <contact_coefficients mu="0" kp="1000.0" kd="1.0"/>

Commit message: Added joint config file and changed structure of sizes config file.

File: urdf_l2/urdf/manip.urdf.xacro (robot description, xacro)
@@ -13,17 +13,4 @@
   <xacro:property name="j3" value="fixed"/>
 </xacro:if>
-<!-- Parametry DH -->
-<xacro:arg name="a1" default="0.5"/>
-<xacro:arg name="a2" default="0.5"/>
-<xacro:arg name="a3" default="0.5"/>
-<xacro:arg name="d1" default="0.5"/>
-<xacro:arg name="d2" default="0.5"/>
-<xacro:arg name="d3" default="0.5"/>
-<xacro:arg name="alpha1" default="0.5"/>
-<xacro:arg name="alpha2" default="0.5"/>
-<xacro:arg name="alpha3" default="0.5"/>
-<xacro:arg name="t1" default="0.5"/>
-<xacro:arg name="t2" default="0.5"/>
-<xacro:arg name="t3" default="0.5"/>
 <link name="base">
   <visual>
@@ -51,14 +38,14 @@
 <link name="el1">
   <visual>
-    <origin xyz="0 0 ${sizes['sizes']['l1']/2}" />
+    <origin xyz="0 0 ${sizes['el1']['l']/2}" />
     <geometry>
-      <cylinder radius="${sizes['sizes']['r1']}" length="${sizes['sizes']['l1']}"/>
+      <cylinder radius="${sizes['el1']['r']}" length="${sizes['el1']['l']}"/>
     </geometry>
     <material name="white"/>
   </visual>
   <collision>
-    <origin xyz="0 0 ${sizes['sizes']['r1']/2}" />
+    <origin xyz="0 0 ${sizes['el1']['r']/2}" />
     <geometry>
-      <cylinder radius="${sizes['sizes']['r1']}" length="${sizes['sizes']['l1']}"/>
+      <cylinder radius="${sizes['el1']['r']}" length="${sizes['el1']['l']}"/>
     </geometry>
     <contact_coefficients mu="0" kp="1000.0" kd="1.0"/>
@@ -68,5 +55,6 @@
   <parent link="el1"/>
   <child link="el2"/>
-  <origin xyz="0 0 ${sizes['sizes']['l1']+0.1}" rpy="0 0 0" />
+  <origin xyz="${joints['el1-el2']['a']} 0 ${sizes['el1']['l']+joints['el1-el2']['d']}"
+    rpy="${joints['el1-el2']['alpha']} 0 ${joints['el1-el2']['t']}" />
   <axis xyz="0 0 1" />
   <limit upper="0" lower="0.0" effort="10" velocity="10" />
@@ -79,7 +67,7 @@
   </inertial>
   <visual>
-    <origin xyz="0 0 ${sizes['sizes']['l2']/2}" rpy="0 0 0" />
+    <origin xyz="0 0 ${sizes['el2']['l']/2}" rpy="0 0 0" />
     <geometry>
-      <cylinder radius="${sizes['sizes']['r2']}" length="${sizes['sizes']['l2']}"/>
+      <cylinder radius="${sizes['el2']['r']}" length="${sizes['el2']['l']}"/>
     </geometry>
     <material name="white">
@@ -88,7 +76,7 @@
   </visual>
   <collision>
-    <origin xyz="0 0 ${sizes['sizes']['l2']/2}" />
+    <origin xyz="0 0 ${sizes['el2']['l']/2}" />
     <geometry>
-      <cylinder radius="${sizes['sizes']['r2']}" length="${sizes['sizes']['l2']}"/>
+      <cylinder radius="${sizes['el2']['r']}" length="${sizes['el2']['l']}"/>
     </geometry>
     <contact_coefficients mu="0" kp="1000.0" kd="1.0"/>
@@ -98,5 +86,6 @@
   <parent link="el2"/>
   <child link="el3"/>
-  <origin xyz="0 0 ${sizes['sizes']['l2']/2}" rpy="0 0 0" />
+  <origin xyz="${joints['el2-el3']['a']} 0 ${sizes['el2']['l']/2+joints['el2-el3']['d']}"
+    rpy="${joints['el2-el3']['alpha']} 0 ${joints['el2-el3']['t']}" />
   <axis xyz="0 0 1" />
   <limit upper="0" lower="0.0" effort="10" velocity="10" />
@@ -109,7 +98,7 @@
   </inertial>
   <visual>
-    <origin xyz="${sizes['sizes']['r2']+sizes['sizes']['r3']} 0 0"/>
+    <origin xyz="${sizes['el2']['r']+sizes['el3']['r']} 0 0"/>
     <geometry>
-      <cylinder radius="${sizes['sizes']['r3']}" length="${sizes['sizes']['l3']}"/>
+      <cylinder radius="${sizes['el3']['r']}" length="${sizes['el3']['l']}"/>
     </geometry>
     <material name="white">
@@ -118,7 +107,7 @@
   </visual>
   <collision>
-    <origin xyz="${sizes['sizes']['r2']+sizes['sizes']['r3']} 0 0"/>
+    <origin xyz="${sizes['el2']['r']+sizes['el3']['r']} 0 0"/>
     <geometry>
-      <cylinder radius="${sizes['sizes']['r3']}" length="${sizes['sizes']['l3']}"/>
+      <cylinder radius="${sizes['el3']['r']}" length="${sizes['el3']['l']}"/>
     </geometry>
     <contact_coefficients mu="0" kp="1000.0" kd="1.0"/>
@@ -128,5 +117,6 @@
   <parent link="el3"/>
   <child link="tool"/>
-  <origin xyz="${2*sizes['sizes']['r3']} 0 0" rpy="0 0 0" />
+  <origin xyz="${2*sizes['el3']['r']+joints['el3-tool']['a']} 0 ${joints['el3-tool']['d']}"
+    rpy="${joints['el3-tool']['alpha']} 0 ${joints['el3-tool']['t']}" />
   <axis xyz="0 0 1" />
   <limit upper="0" lower="0.0" effort="10" velocity="10" />
@@ -139,7 +129,7 @@
   </inertial>
   <visual>
-    <origin xyz="${sizes['sizes']['l4']/2+sizes['sizes']['r3']} 0 0" />
+    <origin xyz="${sizes['tool']['l']/2+sizes['el3']['r']} 0 0" />
     <geometry>
-      <box size="${sizes['sizes']['l4']} ${sizes['sizes']['aa4']} ${sizes['sizes']['aa4']}"/>
+      <box size="${sizes['tool']['l']} ${sizes['tool']['aa']} ${sizes['tool']['aa']}"/>
     </geometry>
     <material name="white">
@@ -148,7 +138,7 @@
   </visual>
   <collision>
-    <origin xyz="${sizes['sizes']['l4']/2+sizes['sizes']['r3']} 0 0" />
+    <origin xyz="${sizes['tool']['l']/2+sizes['el3']['r']} 0 0" />
     <geometry>
-      <box size="${sizes['sizes']['l4']} ${sizes['sizes']['aa4']} ${sizes['sizes']['aa4']}"/>
+      <box size="${sizes['tool']['l']} ${sizes['tool']['aa']} ${sizes['tool']['aa']}"/>
     </geometry>
     <contact_coefficients mu="0" kp="1000.0" kd="1.0"/>
