Commit message: DH to RPY conversion and parameter reorganisation.

File: dkin_l3/urdf/manip.urdf.xacro (robot description, xacro)
@@ -1,8 +1,10 @@
 <?xml version="1.0" encoding="utf-8"?>
 <robot xmlns:xacro="http://www.ros.org/wiki/xacro" name="manip">
-<!-- Rozmiary czlonow -->
-<xacro:property name="sizes" value="${load_yaml('sizes.yaml')}"/>
+<!-- Parametry czlonow -->
+<xacro:property name="links" value="${load_yaml('links.yaml')}"/>
 <!-- Stawy -->
 <xacro:property name="joints" value="${load_yaml('joints.yaml')}"/>
+<!-- Parametry stawow -->
+<xacro:property name="xyz_rpy" value="${load_yaml('xyz_rpy.yaml')}"/>
 <xacro:property name="j1" value="prismatic"/>
 <xacro:property name="j2" value="revolute"/>
@@ -17,5 +19,8 @@
     <origin xyz="0 0 0.1" />
     <geometry>
-      <box size="1 1 0.2"/>
+      <box size="
+        ${links['base']['l']}
+        ${links['base']['l']}
+        ${links['base']['w']}" />
     </geometry>
     <material name="white">
@@ -26,5 +31,8 @@
     <origin xyz="0 0 0.1" />
     <geometry>
-      <box size="1 1 0.2"/>
+      <box size="
+        ${links['base']['l']}
+        ${links['base']['l']}
+        ${links['base']['w']}" />
     </geometry>
     <contact_coefficients mu="0" kp="1000.0" kd="1.0"/>
@@ -34,18 +42,25 @@
   <parent link="base"/>
   <child link="el1"/>
-  <origin xyz="${joints['el1-el2']['a']} 0 0.2" rpy="0 0 0" />
+  <origin xyz="
+    ${xyz_rpy['base-el1']['x']}
+    ${xyz_rpy['base-el1']['y']}
+    ${xyz_rpy['base-el1']['z']}"
+    rpy="
+    ${xyz_rpy['base-el1']['roll']}
+    ${xyz_rpy['base-el1']['pitch']}
+    ${xyz_rpy['base-el1']['yaw']}" />
 </joint>
 <link name="el1">
   <visual>
-    <origin xyz="0 0 ${sizes['el1']['l']/2}" />
+    <origin xyz="0 0 ${links['el1']['l']/2}" />
     <geometry>
-      <cylinder radius="${sizes['el1']['r']}" length="${sizes['el1']['l']}"/>
+      <cylinder radius="${links['el1']['r']}" length="${links['el1']['l']}"/>
     </geometry>
     <material name="white"/>
   </visual>
   <collision>
-    <origin xyz="0 0 ${sizes['el1']['r']/2}" />
+    <origin xyz="0 0 ${links['el1']['r']/2}" />
     <geometry>
-      <cylinder radius="${sizes['el1']['r']}" length="${sizes['el1']['l']}"/>
+      <cylinder radius="${links['el1']['r']}" length="${links['el1']['l']}"/>
     </geometry>
     <contact_coefficients mu="0" kp="1000.0" kd="1.0"/>
@@ -55,6 +70,12 @@
   <parent link="el1"/>
   <child link="el2"/>
-  <origin xyz="${joints['el2-el3']['a']} 0 ${sizes['el1']['l']+joints['el1-el2']['d']}"
-    rpy="${joints['el1-el2']['alpha']} 0 ${joints['el1-el2']['t']}" />
+  <origin xyz="
+    ${xyz_rpy['el1-el2']['x']}
+    ${xyz_rpy['el1-el2']['y']}
+    ${xyz_rpy['el1-el2']['z']}"
+  rpy="
+    ${xyz_rpy['el1-el2']['roll']}
+    ${xyz_rpy['el1-el2']['pitch']}
+    ${xyz_rpy['el1-el2']['yaw']}" />
   <axis xyz="0 0 1" />
   <limit upper="0" lower="0.0" effort="10" velocity="10" />
@@ -67,7 +88,7 @@
   </inertial>
   <visual>
-    <origin xyz="0 0 ${sizes['el2']['l']/2}" rpy="0 0 0" />
+    <origin xyz="0 0 ${links['el2']['l']/2}" rpy="0 0 0" />
     <geometry>
-      <cylinder radius="${sizes['el2']['r']}" length="${sizes['el2']['l']}"/>
+      <cylinder radius="${links['el2']['r']}" length="${links['el2']['l']}"/>
     </geometry>
     <material name="white">
@@ -76,7 +97,7 @@
   </visual>
   <collision>
-    <origin xyz="0 0 ${sizes['el2']['l']/2}" />
+    <origin xyz="0 0 ${links['el2']['l']/2}" />
     <geometry>
-      <cylinder radius="${sizes['el2']['r']}" length="${sizes['el2']['l']}"/>
+      <cylinder radius="${links['el2']['r']}" length="${links['el2']['l']}"/>
     </geometry>
     <contact_coefficients mu="0" kp="1000.0" kd="1.0"/>
@@ -86,6 +107,12 @@
   <parent link="el2"/>
   <child link="el3"/>
-  <origin xyz="0 0 ${sizes['el2']['l']/2+joints['el2-el3']['d']}"
-    rpy="${joints['el2-el3']['alpha']} 0 ${joints['el2-el3']['t']}" />
+  <origin xyz="
+    ${xyz_rpy['el2-el3']['x']}
+    ${xyz_rpy['el2-el3']['y']}
+    ${xyz_rpy['el2-el3']['z']}"
+    rpy="
+    ${xyz_rpy['el2-el3']['roll']}
+    ${xyz_rpy['el2-el3']['pitch']}
+    ${xyz_rpy['el2-el3']['yaw']}" />
   <axis xyz="0 0 1" />
   <limit upper="0" lower="0.0" effort="10" velocity="10" />
@@ -98,7 +125,7 @@
   </inertial>
   <visual>
-    <origin xyz="${joints['el3-tool']['a']} 0 0"/>
+    <origin xyz="${links['el3']['a']} 0 0"/>
     <geometry>
-      <cylinder radius="${sizes['el3']['r']}" length="${sizes['el3']['l']}"/>
+      <cylinder radius="${links['el3']['r']}" length="${links['el3']['l']}"/>
     </geometry>
     <material name="white">
@@ -107,7 +134,7 @@
   </visual>
   <collision>
-    <origin xyz="${sizes['el2']['r']+sizes['el3']['r']} 0 0"/>
+    <origin xyz="${links['el2']['r']+links['el3']['r']} 0 0"/>
     <geometry>
-      <cylinder radius="${sizes['el3']['r']}" length="${sizes['el3']['l']}"/>
+      <cylinder radius="${links['el3']['r']}" length="${links['el3']['l']}"/>
     </geometry>
     <contact_coefficients mu="0" kp="1000.0" kd="1.0"/>
@@ -117,6 +144,12 @@
   <parent link="el3"/>
   <child link="tool"/>
-  <origin xyz="${joints['el3-tool']['a']} 0 0"
-    rpy="${joints['el3-tool']['alpha']} 0 ${joints['el3-tool']['t']}" />
+  <origin xyz="
+    ${xyz_rpy['el3-tool']['x']}
+    ${xyz_rpy['el3-tool']['y']}
+    ${xyz_rpy['el3-tool']['z']}"
+  rpy="
+    ${xyz_rpy['el3-tool']['roll']}
+    ${xyz_rpy['el3-tool']['pitch']}
+    ${xyz_rpy['el3-tool']['yaw']}" />
   <axis xyz="0 0 1" />
   <limit upper="0" lower="0.0" effort="10" velocity="10" />
@@ -129,7 +162,7 @@
   </inertial>
   <visual>
-    <origin xyz="${sizes['tool']['l']/2+sizes['el3']['r']} 0 0" />
+    <origin xyz="${links['tool']['l']/2+links['el3']['r']} 0 0" />
     <geometry>
-      <box size="${sizes['tool']['l']} ${sizes['tool']['aa']} ${sizes['tool']['aa']}"/>
+      <box size="${links['tool']['l']} ${links['tool']['aa']} ${links['tool']['aa']}"/>
     </geometry>
     <material name="white">
@@ -138,7 +171,7 @@
   </visual>
   <collision>
-    <origin xyz="${sizes['tool']['l']/2+sizes['el3']['r']} 0 0" />
+    <origin xyz="${links['tool']['l']/2+links['el3']['r']} 0 0" />
     <geometry>
-      <box size="${sizes['tool']['l']} ${sizes['tool']['aa']} ${sizes['tool']['aa']}"/>
+      <box size="${links['tool']['l']} ${links['tool']['aa']} ${links['tool']['aa']}"/>
     </geometry>
     <contact_coefficients mu="0" kp="1000.0" kd="1.0"/>
