Commit message: Created communication structures

File: ikin_l5/urdf/manip.urdf.xacro (robot description, xacro)
@@ -28,14 +28,4 @@
     </material>
   </visual>
-  <collision>
-    <origin xyz="0 0 0.1" />
-    <geometry>
-      <box size="
-        ${links['base']['l']}
-        ${links['base']['l']}
-        ${links['base']['w']}" />
-    </geometry>
-    <contact_coefficients mu="0" kp="1000.0" kd="1.0"/>
-  </collision>
 </link>
 <joint name="base-el1" type="fixed">
@@ -59,11 +49,4 @@
     <material name="white"/>
   </visual>
-  <collision>
-    <origin xyz="0 0 ${links['el1']['r']/2}" />
-    <geometry>
-      <cylinder radius="${links['el1']['r']}" length="${links['el1']['l']}"/>
-    </geometry>
-    <contact_coefficients mu="0" kp="1000.0" kd="1.0"/>
-  </collision>
 </link>
 <joint name="el1-el2" type="${j1}">
@@ -96,11 +79,4 @@
     </material>
   </visual>
-  <collision>
-    <origin xyz="0 0 ${links['el2']['l']/2}" />
-    <geometry>
-      <cylinder radius="${links['el2']['r']}" length="${links['el2']['l']}"/>
-    </geometry>
-    <contact_coefficients mu="0" kp="1000.0" kd="1.0"/>
-  </collision>
 </link>
 <joint name="el2-el3" type="${j2}">
@@ -133,11 +109,4 @@
     </material>
   </visual>
-  <collision>
-    <origin xyz="${links['el2']['r']+links['el3']['r']} 0 0"/>
-    <geometry>
-      <cylinder radius="${links['el3']['r']}" length="${links['el3']['l']}"/>
-    </geometry>
-    <contact_coefficients mu="0" kp="1000.0" kd="1.0"/>
-  </collision>
 </link>
 <joint name="el3-tool" type="${j3}">
@@ -170,11 +139,4 @@
     </material>
   </visual>
-  <collision>
-    <origin xyz="${links['tool']['l']/2+links['el3']['r']} 0 0" />
-    <geometry>
-      <box size="${links['tool']['l']} ${links['tool']['aa']} ${links['tool']['aa']}"/>
-    </geometry>
-    <contact_coefficients mu="0" kp="1000.0" kd="1.0"/>
-  </collision>
 </link>
 </robot>

Commit message: Fixed model

File: ikin_l5/urdf/manip.urdf.xacro (robot description, xacro)
@@ -94,4 +94,20 @@
   <limit upper="0" lower="0.0" effort="10" velocity="10" />
 </joint>
+<joint name="el2-el3-fill" type="fixed">
+  <parent link="el3"/>
+  <child link="2-3-fill"/>
+  <origin xyz="${links['el3']['a']/2} 0 0" rpy="0 1.57 0"/>
+</joint>
+<link name="2-3-fill">
+  <visual>
+    <origin xyz="0 0 0"/>
+    <geometry>
+      <cylinder radius="${links['tool']['aa']/2}" length="${links['el3']['a']}"/>
+    </geometry>
+    <material name="white">
+      <color rgba="1 1 1 1" />
+    </material>
+  </visual>
+</link>
 <link name="el3">
   <inertial>
@@ -140,3 +156,19 @@
   </visual>
 </link>
+<joint name="tool-toolend" type="fixed">
+  <parent link="tool"/>
+  <child link="toolend"/>
+  <origin xyz="${links['tool']['l']+links['el3']['r']} 0 0" rpy="0 0 0"/>
+</joint>
+<link name="toolend">
+  <visual>
+    <origin xyz="0 0 0"/>
+    <geometry>
+      <sphere radius="${links['tool']['aa']/2}"/>
+    </geometry>
+    <material name="white">
+      <color rgba="1 1 1 1" />
+    </material>
+  </visual>
+</link>
 </robot>
